File: KiCad/Gas_Sensor.kicad_pcb (KiCad board)
At the start: 2 copper layers, 59.1 x 54.6 mm, 18 parts, among them J1 Conn_01x07, Q1 IRF520, SW1 SW_SPDT, U1 Capteur_Gaz, U3 MCP41100

Commit message: README update
Parts:
- moved R7 7.41 mm to (71.1, 62.2)
Routing:
- net +12V: track 16.6 -> 6.40 mm, vias 2 -> 0
- net SW_12V: track 27.2 -> 33.6 mm

Commit message: Update README
Other:
- board text added: "Heusse Holmes"
Changed lines of the file:
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@@
   (gr_line (start 39.37 16.51) (end 92.71 16.51)
     (stroke (width 0.1) (type default)) (layer "Edge.Cuts"))
+  (gr_text "Heusse Holmes" (at 45.0088 47.3964 90) (layer "B.Cu" knockout)
+    (effects (font (size 1.2 1.2) (thickness 0.3) bold) (justify left bottom mirror))
+  )
   (segment (start 84.5955 26.67) (end 91.44 26.67) (width 0.8) (layer "F.Cu") (net 1))
   (segment (start 91.44 26.67) (end 92.075 27.305) (width 0.8) (layer "F.Cu") (net 1))
